File: eagle/thesis.sch (EAGLE design)
At the start: 6 parts, among them U1 ITG-3200, U2 ADXL362

Commit message: made changes to eagle files
Parts:
- added VGA1: VGA-F90S, VideoConnectors:VGA-F90S
Connections:
- removed net N$12: U$1.10, U2.!CS
- removed net N$13: U$1.5V_ICSP, U2.GND
- removed net N$2: U$1.SCK_ICSP, U$2.CLK, U2.SCLK
- removed net N$3: U$1.MISO_ICSP, U$2.DO, U2.MISO
- removed net N$4: U$1.MOSI_ICSP, U$2.DI, U2.MOSI
- removed net N$5: U$1.53, U$2./CS
- removed net N$7: U$1.SDA1, U1.SDA
- removed net N$8: U$1.SCL1, U1.SCL
- net N$1: now also U2.GND; no longer U$1.GND_1, U$2.VDD
- net N$6: no longer U$1.3V3, U$2.VSS, U2.VDDIO, U2.VS
Changed lines of the file:
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@@
 <part name="C2" library="SparkFun-Capacitors" deviceset="CAP" device="KIT" value="2.2nF"/>
 <part name="U2" library="SparkFun-Sensors" deviceset="ADXL362" device="" value="ADXL362"/>
+<part name="VGA1" library="VideoConnectors" deviceset="VGA-*" device="F90S"/>
 </parts>
 <sheets>
@@
 <instance part="C2" gate="G$1" x="10.16" y="109.22"/>
 <instance part="U2" gate="G$1" x="-142.24" y="132.08" rot="R180"/>
+<instance part="VGA1" gate="G$1" x="-106.68" y="170.18"/>
 </instances>
 <busses>
 </busses>
 <nets>
-<net name="N$2" class="0">
-<segment>
-<pinref part="U$2" gate="G$1" pin="CLK"/>
-<wire x1="-134.62" y1="99.06" x2="-104.14" y2="99.06" width="0.1524" layer="91"/>
-<wire x1="-104.14" y1="99.06" x2="-104.14" y2="127" width="0.1524" layer="91"/>
-<pinref part="U$1" gate="G$1" pin="SCK_ICSP"/>
-<wire x1="-104.14" y1="127" x2="-104.14" y2="129.54" width="0.1524" layer="91"/>
-<wire x1="-104.14" y1="129.54" x2="-93.98" y2="129.54" width="0.1524" layer="91"/>
-<pinref part="U2" gate="G$1" pin="SCLK"/>
-<wire x1="-127" y1="127" x2="-104.14" y2="127" width="0.1524" layer="91"/>
-<junction x="-104.14" y="127"/>
-</segment>
-</net>
-<net name="N$3" class="0">
-<segment>
-<pinref part="U$1" gate="G$1" pin="MISO_ICSP"/>
-<wire x1="-93.98" y1="127" x2="-101.6" y2="127" width="0.1524" layer="91"/>
-<wire x1="-101.6" y1="127" x2="-101.6" y2="93.98" width="0.1524" layer="91"/>
-<pinref part="U$2" gate="G$1" pin="DO"/>
-<wire x1="-134.62" y1="93.98" x2="-101.6" y2="93.98" width="0.1524" layer="91"/>
-<pinref part="U2" gate="G$1" pin="MISO"/>
-<wire x1="-127" y1="132.08" x2="-93.98" y2="132.08" width="0.1524" layer="91"/>
-<wire x1="-93.98" y1="132.08" x2="-93.98" y2="127" width="0.1524" layer="91"/>
-<junction x="-93.98" y="127"/>
-</segment>
-</net>
-<net name="N$4" class="0">
-<segment>
-<pinref part="U$2" gate="G$1" pin="DI"/>
-<wire x1="-134.62" y1="104.14" x2="-99.06" y2="104.14" width="0.1524" layer="91"/>
-<wire x1="-99.06" y1="104.14" x2="-99.06" y2="124.46" width="0.1524" layer="91"/>
-<pinref part="U$1" gate="G$1" pin="MOSI_ICSP"/>
-<wire x1="-93.98" y1="124.46" x2="-99.06" y2="124.46" width="0.1524" layer="91"/>
-<pinref part="U2" gate="G$1" pin="MOSI"/>
-<wire x1="-127" y1="129.54" x2="-106.68" y2="129.54" width="0.1524" layer="91"/>
-<wire x1="-106.68" y1="129.54" x2="-106.68" y2="124.46" width="0.1524" layer="91"/>
-<wire x1="-106.68" y1="124.46" x2="-93.98" y2="124.46" width="0.1524" layer="91"/>
-<junction x="-93.98" y="124.46"/>
-</segment>
-</net>
-<net name="N$5" class="0">
-<segment>
-<pinref part="U$2" gate="G$1" pin="/CS"/>
-<wire x1="-134.62" y1="106.68" x2="-116.84" y2="106.68" width="0.1524" layer="91"/>
-<wire x1="-116.84" y1="106.68" x2="-116.84" y2="43.18" width="0.1524" layer="91"/>
-<wire x1="-116.84" y1="43.18" x2="10.16" y2="43.18" width="0.1524" layer="91"/>
-<wire x1="10.16" y1="43.18" x2="10.16" y2="58.42" width="0.1524" layer="91"/>
-<pinref part="U$1" gate="G$1" pin="53"/>
-<wire x1="10.16" y1="58.42" x2="-22.86" y2="58.42" width="0.1524" layer="91"/>
-</segment>
-</net>
-<net name="N$1" class="0">
-<segment>
-<pinref part="U$2" gate="G$1" pin="VDD"/>
-<wire x1="-134.62" y1="101.6" x2="-111.76" y2="101.6" width="0.1524" layer="91"/>
-<wire x1="-111.76" y1="101.6" x2="-111.76" y2="63.5" width="0.1524" layer="91"/>
-<pinref part="U$1" gate="G$1" pin="GND_1"/>
-<wire x1="-111.76" y1="63.5" x2="-93.98" y2="63.5" width="0.1524" layer="91"/>
-</segment>
-</net>
-<net name="N$7" class="0">
-<segment>
-<pinref part="U1" gate="G$1" pin="SDA"/>
-<wire x1="50.8" y1="129.54" x2="66.04" y2="129.54" width="0.1524" layer="91"/>
-<wire x1="66.04" y1="129.54" x2="66.04" y2="154.94" width="0.1524" layer="91"/>
-<wire x1="66.04" y1="154.94" x2="-81.28" y2="154.94" width="0.1524" layer="91"/>
-<pinref part="U$1" gate="G$1" pin="SDA1"/>
-<wire x1="-81.28" y1="154.94" x2="-81.28" y2="142.24" width="0.1524" layer="91"/>
-</segment>
-</net>
-<net name="N$8" class="0">
-<segment>
-<pinref part="U1" gate="G$1" pin="SCL"/>
-<wire x1="50.8" y1="124.46" x2="73.66" y2="124.46" width="0.1524" layer="91"/>
-<wire x1="73.66" y1="124.46" x2="73.66" y2="157.48" width="0.1524" layer="91"/>
-<pinref part="U$1" gate="G$1" pin="SCL1"/>
-<wire x1="73.66" y1="157.48" x2="-83.82" y2="157.48" width="0.1524" layer="91"/>
-<wire x1="-83.82" y1="157.48" x2="-83.82" y2="142.24" width="0.1524" layer="91"/>
-</segment>
-</net>
 <net name="N$10" class="0">
 <segment>
@@
 <net name="N$6" class="0">
 <segment>
-<pinref part="U$1" gate="G$1" pin="3V3"/>
-<wire x1="-109.22" y1="68.58" x2="-93.98" y2="68.58" width="0.1524" layer="91"/>
-<pinref part="U$2" gate="G$1" pin="VSS"/>
-<wire x1="-134.62" y1="96.52" x2="-109.22" y2="96.52" width="0.1524" layer="91"/>
-<wire x1="-109.22" y1="96.52" x2="-109.22" y2="68.58" width="0.1524" layer="91"/>
-<wire x1="-109.22" y1="152.4" x2="-109.22" y2="96.52" width="0.1524" layer="91"/>
-<junction x="-109.22" y="96.52"/>
 <pinref part="U1" gate="G$1" pin="VDD"/>
 <wire x1="22.86" y1="129.54" x2="15.24" y2="129.54" width="0.1524" layer="91"/>
 <wire x1="15.24" y1="129.54" x2="15.24" y2="152.4" width="0.1524" layer="91"/>
-<wire x1="15.24" y1="152.4" x2="-109.22" y2="152.4" width="0.1524" layer="91"/>
 <pinref part="U1" gate="G$1" pin="VLOGIC"/>
 <wire x1="22.86" y1="124.46" x2="15.24" y2="124.46" width="0.1524" layer="91"/>
@@
 <wire x1="60.96" y1="109.22" x2="60.96" y2="152.4" width="0.1524" layer="91"/>
 <wire x1="60.96" y1="152.4" x2="15.24" y2="152.4" width="0.1524" layer="91"/>
-<junction x="15.24" y="152.4"/>
-<wire x1="-109.22" y1="152.4" x2="-165.1" y2="152.4" width="0.1524" layer="91"/>
-<wire x1="-165.1" y1="152.4" x2="-165.1" y2="129.54" width="0.1524" layer="91"/>
-<junction x="-109.22" y="152.4"/>
-<pinref part="U2" gate="G$1" pin="VDDIO"/>
-<wire x1="-165.1" y1="129.54" x2="-165.1" y2="127" width="0.1524" layer="91"/>
-<wire x1="-165.1" y1="127" x2="-157.48" y2="127" width="0.1524" layer="91"/>
-<pinref part="U2" gate="G$1" pin="VS"/>
-<wire x1="-157.48" y1="129.54" x2="-165.1" y2="129.54" width="0.1524" layer="91"/>
-<junction x="-165.1" y="129.54"/>
 </segment>
 </net>
@@
 </segment>
 </net>
-<net name="N$13" class="0">
+<net name="N$1" class="0">
 <segment>
 <pinref part="U2" gate="G$1" pin="GND"/>
-<wire x1="-157.48" y1="137.16" x2="-160.02" y2="137.16" width="0.1524" layer="91"/>
-<wire x1="-160.02" y1="137.16" x2="-160.02" y2="142.24" width="0.1524" layer="91"/>
-<wire x1="-160.02" y1="142.24" x2="-104.14" y2="142.24" width="0.1524" layer="91"/>
-<wire x1="-104.14" y1="142.24" x2="-104.14" y2="134.62" width="0.1524" layer="91"/>
-<pinref part="U$1" gate="G$1" pin="5V_ICSP"/>
-<wire x1="-104.14" y1="134.62" x2="-93.98" y2="134.62" width="0.1524" layer="91"/>
+<wire x1="-157.48" y1="137.16" x2="-167.64" y2="137.16" width="0.1524" layer="91"/>
 </segment>
 </net>
-<net name="N$12" class="0">
-<segment>
-<pinref part="U2" gate="G$1" pin="!CS"/>
-<wire x1="-127" y1="134.62" x2="-114.3" y2="134.62" width="0.1524" layer="91"/>
-<wire x1="-114.3" y1="134.62" x2="-114.3" y2="165.1" width="0.1524" layer="91"/>
-<pinref part="U$1" gate="G$1" pin="10"/>
-<wire x1="-114.3" y1="165.1" x2="-40.64" y2="165.1" width="0.1524" layer="91"/>
-<wire x1="-40.64" y1="165.1" x2="-40.64" y2="142.24" width="0.1524" layer="91"/>
-</segment>
-</net>
