File: eagle/satellite.brd (EAGLE design)
At the start: 100 x 80 mm, 5 parts

Commit message: changes to eagle files
Parts:
- removed VGA1: VGA-F90S, VideoConnectors:DB-15-F90+SHIELD-SMALL_PADS
- added JP10, JP8, JP9: (no value), pinhead:1X03
- added JP5, JP6: (no value), te-con-rj50:1X05
- added JP7: (no value), pinhead:1X02
- added R1: 4.7K, rcl:0204/5
- added U$1: TECONN5558065-1, te-con-rj50:RJ50
Connections:
- removed net CS1: VGA1.6
- removed net CS2: JP2.6, VGA1.7
- removed net CS3: JP3.6, VGA1.8
- removed net CS4: JP4.6, VGA1.9
- new net 33V: JP5.5
- new net BR: JP1.5, JP2.5, JP3.5, JP4.5, JP7.2, R1.2
- new net RX: JP1.2, JP2.2, JP3.2, JP4.2, JP5.2
- new net SCL: JP10.1, JP6.2
- new net SDA: JP10.2, JP6.1
- new net TX: JP1.3, JP2.3, JP3.3, JP4.3, JP5.1
- net 5V: now also JP1.1, JP2.1, JP3.1, JP4.1, JP5.4, R1.1; no longer JP1.2, JP2.2, JP3.2, JP4.2, VGA1.2
- net GND: now also JP1.4, JP2.4, JP2.6, JP3.4, JP3.6, JP4.4, JP4.6, JP5.3, JP7.1; no longer JP1.1, JP2.1, JP3.1, JP4.1, VGA1.1
- net MISO: now also JP6.5, JP9.1; no longer JP1.4, JP2.4, JP3.4, JP4.4, VGA1.3
- net MOSI: now also JP6.4, JP9.2; no longer JP1.3, JP2.3, JP3.3, JP4.3, VGA1.4
- net SCK: now also JP6.3, JP9.3; no longer JP1.5, JP2.5, JP3.5, JP4.5, VGA1.5
Routing:
- net MOSI: track 204.6 -> 0.00 mm
- net TX: track 0.00 -> 204.4 mm
- net GND: track 148.0 -> 346.8 mm, vias 0 -> 2
- net RX: track 0.00 -> 179.3 mm, vias 0 -> 1
- net MISO: track 170.4 -> 0.00 mm
- net SCK: track 134.4 -> 0.00 mm
- net BR: track 0.00 -> 134.1 mm
- net CS3: track 91.5 -> 0.00 mm
- net CS2: track 67.9 -> 0.00 mm
- net 5V: track 179.9 -> 147.2 mm, vias 1 -> 0
- net CS4: track 31.6 -> 0.00 mm, vias 2 -> 0
