File: eagle/satellite.sch (EAGLE design)
At the start: 5 parts

Commit message: changes to eagle files
Parts:
- removed VGA1: VGA-F90S, VideoConnectors:VGA-F90S
- added JP10, JP8, JP9: (no value), pinhead:PINHD-1X3
- added JP5, JP6: (no value), te-con-rj50:PINHD-1X5
- added JP7: (no value), pinhead:PINHD-1X2
- added R1: 4.7K, rcl:R-US_0204/5
- added U$1: TECONN5558065-1, te-con-rj50:TECONN5558065-1
Connections:
- removed net CS1: VGA1G$1.VGA-R-
- removed net CS2: JP2.6, VGA1G$1.VGA-G-
- removed net CS3: JP3.6, VGA1G$1.VGA-B-
- removed net CS4: JP4.6, VGA1G$1.+5V
- new net 33V: JP5.5
- new net BR: JP1.5, JP2.5, JP3.5, JP4.5, JP7.2, R1.2
- new net RX: JP1.2, JP2.2, JP3.2, JP4.2, JP5.2
- new net SCL: JP10.1, JP6.2
- new net SDA: JP10.2, JP6.1
- new net TX: JP1.3, JP2.3, JP3.3, JP4.3, JP5.1
- net 5V: now also JP1.1, JP2.1, JP3.1, JP4.1, JP5.4, R1.1; no longer JP1.2, JP2.2, JP3.2, JP4.2, VGA1G$1.VGA-G
- net GND: now also JP1.4, JP2.4, JP2.6, JP3.4, JP3.6, JP4.4, JP4.6, JP5.3, JP7.1; no longer JP1.1, JP2.1, JP3.1, JP4.1, VGA1G$1.VGA-R
- net MISO: now also JP6.5, JP9.1; no longer JP1.4, JP2.4, JP3.4, JP4.4, VGA1G$1.VGA-B
- net MOSI: now also JP6.4, JP9.2; no longer JP1.3, JP2.3, JP3.3, JP4.3, VGA1G$1.ID2/RES
- net SCK: now also JP6.3, JP9.3; no longer JP1.5, JP2.5, JP3.5, JP4.5, VGA1G$1.GND@0
