File: eagle/magBoard.brd (EAGLE design)
At the start: 43.2 x 41.4 mm, 9 parts, among them J1 RJ11-6PTH, U3 MAX3232PTH

Commit message: wrote a bunch and added references and pictures
Connections:
- net RS232IN renamed RS232DI
Routing:
- net RS232DI: track 27.6 -> 0.00 mm
- net GND: track 67.7 -> 60.5 mm
- net RS232DO: track 28.2 -> 25.9 mm
Changed lines of the file:
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@@
 </signal>
 <signal name="GND">
-<contactref element="U3" pad="15"/>
-<contactref element="HMR2300" pad="5"/>
-<contactref element="C2" pad="2"/>
 <contactref element="C6" pad="2"/>
 <contactref element="J1" pad="6"/>
-<wire x1="23.368" y1="29.337" x2="25.781" y2="31.75" width="0.254" layer="1"/>
 <wire x1="23.368" y1="25.654" x2="23.368" y2="29.337" width="0.254" layer="1"/>
 <wire x1="22.86" y1="25.146" x2="23.368" y2="25.654" width="0.254" layer="1"/>
@@
 <wire x1="15.621" y1="25.654" x2="15.621" y2="25.146" width="0.254" layer="1"/>
 <wire x1="30.988" y1="14.859" x2="24.9555" y2="8.8265" width="0.254" layer="16"/>
-<wire x1="24.9555" y1="8.8265" x2="23.368" y2="7.239" width="0.254" layer="16"/>
 <wire x1="31.496" y1="14.859" x2="30.988" y2="14.859" width="0.254" layer="16"/>
-<wire x1="31.496" y1="14.859" x2="31.6" y2="14.907" width="0.254" layer="16"/>
 <wire x1="2.921" y1="8.89" x2="2.667" y2="9.144" width="0.254" layer="16"/>
 <wire x1="24.892" y1="8.89" x2="2.921" y2="8.89" width="0.254" layer="16"/>
 <wire x1="24.892" y1="8.89" x2="24.9555" y2="8.8265" width="0.254" layer="16"/>
 <wire x1="22.352" y1="8.255" x2="22.352" y2="25.146" width="0.254" layer="1"/>
-<wire x1="23.368" y1="7.239" x2="22.352" y2="8.255" width="0.254" layer="1"/>
-</signal>
-<signal name="RS232IN">
-<contactref element="HMR2300" pad="3"/>
-<contactref element="U3" pad="13"/>
-<wire x1="19.939" y1="5.588" x2="18.288" y2="7.239" width="0.254" layer="16"/>
-<wire x1="26.416" y1="5.588" x2="19.939" y2="5.588" width="0.254" layer="16"/>
-<wire x1="32.893" y1="12.065" x2="26.416" y2="5.588" width="0.254" layer="16"/>
-<wire x1="32.893" y1="20.447" x2="32.893" y2="12.065" width="0.254" layer="16"/>
-<wire x1="31.6" y1="20.447" x2="32.893" y2="20.447" width="0.254" layer="16"/>
+<contactref element="C2" pad="2"/>
+<contactref element="HMR2300" pad="5"/>
+<contactref element="U3" pad="15"/>
+<wire x1="23.368" y1="29.337" x2="25.781" y2="31.75" width="0" layer="19" extent="1-1"/>
+<wire x1="23.368" y1="7.239" x2="22.352" y2="8.255" width="0" layer="19" extent="1-1"/>
+<wire x1="24.9555" y1="8.8265" x2="23.368" y2="7.239" width="0" layer="19" extent="16-16"/>
+<wire x1="31.6" y1="14.907" x2="31.496" y2="14.859" width="0" layer="19" extent="16-16"/>
 </signal>
 <signal name="RS232DO">
 <contactref element="HMR2300" pad="2"/>
-<contactref element="U3" pad="14"/>
-<wire x1="22.479" y1="5.588" x2="20.828" y2="7.239" width="0.254" layer="1"/>
 <wire x1="30.099" y1="5.588" x2="22.479" y2="5.588" width="0.254" layer="1"/>
 <wire x1="30.099" y1="21.717" x2="30.099" y2="5.588" width="0.254" layer="1"/>
 <wire x1="31.496" y1="23.114" x2="30.099" y2="21.717" width="0.254" layer="1"/>
 <wire x1="31.496" y1="23.114" x2="31.6" y2="23.217" width="0.254" layer="1"/>
+<contactref element="U3" pad="14"/>
+<wire x1="20.828" y1="7.239" x2="22.479" y2="5.588" width="0" layer="19" extent="1-1"/>
 </signal>
 <signal name="DO">
@@
 <wire x1="34.544" y1="16.383" x2="34.44" y2="16.297" width="0.254" layer="16"/>
 </signal>
+<signal name="RS232DI">
+<contactref element="U3" pad="13"/>
+<contactref element="HMR2300" pad="3"/>
+<wire x1="18.288" y1="7.239" x2="31.6" y2="20.447" width="0" layer="19" extent="1-1"/>
+</signal>
 </signals>
