File: eagle/satellitev2.sch (EAGLE design)
At the start: 12 parts, among them J1 RJ11-6PTH

Commit message: modified eagle boards and ordered.
Parts:
- renumbered JP1 to BR
Changed lines of the file:
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@@
 <part name="D3" library="SparkFun-DiscreteSemi" deviceset="DIODE" device="PTH"/>
 <part name="D4" library="SparkFun-DiscreteSemi" deviceset="DIODE" device="PTH"/>
-<part name="JP1" library="pinhead" deviceset="PINHD-1X2" device=""/>
+<part name="BR" library="pinhead" deviceset="PINHD-1X2" device=""/>
 <part name="R2" library="rcl" deviceset="R-US_" device="0309/12" value="2.2K"/>
 </parts>
@@
 <instance part="D3" gate="G$1" x="86.36" y="55.88"/>
 <instance part="D4" gate="G$1" x="83.82" y="20.32"/>
-<instance part="JP1" gate="G$1" x="119.38" y="-7.62"/>
+<instance part="BR" gate="G$1" x="119.38" y="-7.62"/>
 <instance part="R2" gate="G$1" x="88.9" y="-7.62"/>
 </instances>
@@
 </segment>
 <segment>
-<pinref part="JP1" gate="G$1" pin="1"/>
+<pinref part="BR" gate="G$1" pin="1"/>
 <wire x1="116.84" y1="-5.08" x2="99.06" y2="-5.08" width="0.1524" layer="91"/>
 <label x="104.14" y="-5.08" size="1.778" layer="95"/>
@@
 </segment>
 <segment>
-<pinref part="JP1" gate="G$1" pin="2"/>
+<pinref part="BR" gate="G$1" pin="2"/>
 <pinref part="R2" gate="G$1" pin="2"/>
 <wire x1="116.84" y1="-7.62" x2="93.98" y2="-7.62" width="0.1524" layer="91"/>

Commit message: in middle of writing for AIAA paper
Parts:
- removed J1: RJ11-6PTH, SparkFun-Connectors:RJ11-6PTH
- added JP1, JP2: (no value), pinhead:PINHD-2X3
- added JP3: (no value), pinhead:PINHD-1X3
- added X1: (no value), con-subd:F15HDV
Connections:
- new net 3V3: JP3.1, X1.6
- new net ACCEL2CS: JP1.5, X1.4
- new net D46: JP2.2, X1.13
- new net D47: JP2.4, X1.14
- new net D48: JP2.6, X1.15
- new net MISO: JP1.1, X1.7
- new net MOSI: JP1.4, X1.3
- new net SCL: JP2.5, X1.12
- new net SCLK: JP1.3, X1.8
- new net SDA: JP2.3, X1.11
- new net TEMPBUS: JP2.1, X1.10
- net 5V: now also JP1.2, X1.1; no longer J1.1
- net GND: now also JP1.6, X1.2; no longer J1.2
- net RX: now also JP3.3, X1.9; no longer J1.3
- net TX: now also JP3.2, X1.5; no longer J1.4
Changed lines of the file:
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@@
 <part name="U$3" library="1x6smdpins" deviceset="1X6SMDPINSB" device=""/>
 <part name="U$4" library="1x6smdpins" deviceset="1X6SMDPINSB" device=""/>
-<part name="J1" library="SparkFun-Connectors" deviceset="RJ11-6" device="PTH"/>
 <part name="R1" library="rcl" deviceset="R-US_" device="0309/12" value="2.2K"/>
 <part name="D1" library="SparkFun-DiscreteSemi" deviceset="DIODE" device="PTH"/>
@@
 <part name="BR" library="pinhead" deviceset="PINHD-1X2" device=""/>
 <part name="R2" library="rcl" deviceset="R-US_" device="0309/12" value="2.2K"/>
+<part name="X1" library="con-subd" deviceset="F15" device="HDV"/>
+<part name="JP1" library="pinhead" deviceset="PINHD-2X3" device=""/>
+<part name="JP2" library="pinhead" deviceset="PINHD-2X3" device=""/>
+<part name="JP3" library="pinhead" deviceset="PINHD-1X3" device=""/>
 </parts>
 <sheets>
@@
 <instance part="U$3" gate="G$1" x="119.38" y="45.72"/>
 <instance part="U$4" gate="G$1" x="119.38" y="12.7"/>
-<instance part="J1" gate="G$1" x="25.4" y="60.96"/>
 <instance part="R1" gate="G$1" x="60.96" y="76.2"/>
 <instance part="D1" gate="G$1" x="-20.32" y="25.4"/>
@@
 <instance part="BR" gate="G$1" x="119.38" y="-7.62"/>
 <instance part="R2" gate="G$1" x="88.9" y="-7.62"/>
+<instance part="X1" gate="-1" x="-12.7" y="60.96"/>
+<instance part="JP1" gate="A" x="38.1" y="53.34"/>
+<instance part="JP2" gate="A" x="48.26" y="38.1"/>
+<instance part="JP3" gate="A" x="48.26" y="17.78"/>
 </instances>
 <busses>
@@
 <net name="5V" class="0">
 <segment>
-<pinref part="J1" gate="G$1" pin="1"/>
-<wire x1="30.48" y1="55.88" x2="45.72" y2="55.88" width="0.1524" layer="91"/>
-</segment>
-<segment>
 <pinref part="R1" gate="G$1" pin="1"/>
 <wire x1="55.88" y1="76.2" x2="43.18" y2="76.2" width="0.1524" layer="91"/>
+<label x="43.18" y="76.2" size="1.778" layer="95"/>
 </segment>
 <segment>
@@
 <label x="91.44" y="15.24" size="1.778" layer="95"/>
 </segment>
+<segment>
+<pinref part="JP1" gate="A" pin="2"/>
+<wire x1="55.88" y1="55.88" x2="43.18" y2="55.88" width="0.1524" layer="91"/>
+<label x="48.26" y="55.88" size="1.778" layer="95"/>
+</segment>
+<segment>
+<pinref part="X1" gate="-1" pin="1"/>
+<wire x1="-20.32" y1="68.58" x2="-27.94" y2="68.58" width="0.1524" layer="91"/>
+<label x="-27.94" y="68.58" size="1.778" layer="95"/>
+</segment>
 </net>
 <net name="GND" class="0">
-<segment>
-<pinref part="J1" gate="G$1" pin="2"/>
-<wire x1="30.48" y1="58.42" x2="45.72" y2="58.42" width="0.1524" layer="91"/>
-</segment>
 <segment>
 <pinref part="U$1" gate="G$1" pin="P$1"/>
@@
 <label x="96.52" y="53.34" size="1.778" layer="95"/>
 </segment>
+<segment>
+<pinref part="JP1" gate="A" pin="6"/>
+<wire x1="55.88" y1="50.8" x2="43.18" y2="50.8" width="0.1524" layer="91"/>
+<label x="48.26" y="50.8" size="1.778" layer="95"/>
+</segment>
+<segment>
+<pinref part="X1" gate="-1" pin="2"/>
+<wire x1="-20.32" y1="66.04" x2="-27.94" y2="66.04" width="0.1524" layer="91"/>
+<label x="-27.94" y="66.04" size="1.778" layer="95"/>
+</segment>
 </net>
 <net name="RX" class="0">
-<segment>
-<pinref part="J1" gate="G$1" pin="3"/>
-<wire x1="30.48" y1="60.96" x2="45.72" y2="60.96" width="0.1524" layer="91"/>
-</segment>
 <segment>
 <pinref part="U$1" gate="G$1" pin="P$5"/>
@@
 <label x="96.52" y="58.42" size="1.778" layer="95"/>
 </segment>
+<segment>
+<pinref part="JP3" gate="A" pin="3"/>
+<wire x1="38.1" y1="15.24" x2="45.72" y2="15.24" width="0.1524" layer="91"/>
+<label x="38.1" y="15.24" size="1.778" layer="95"/>
+</segment>
+<segment>
+<pinref part="X1" gate="-1" pin="9"/>
+<wire x1="2.54" y1="68.58" x2="-5.08" y2="68.58" width="0.1524" layer="91"/>
+<label x="-2.54" y="68.58" size="1.778" layer="95"/>
+</segment>
 </net>
 <net name="TX" class="0">
-<segment>
-<pinref part="J1" gate="G$1" pin="4"/>
-<wire x1="30.48" y1="63.5" x2="45.72" y2="63.5" width="0.1524" layer="91"/>
-</segment>
 <segment>
 <pinref part="R1" gate="G$1" pin="2"/>
 <wire x1="66.04" y1="76.2" x2="78.74" y2="76.2" width="0.1524" layer="91"/>
+<label x="73.66" y="76.2" size="1.778" layer="95"/>
 </segment>
 <segment>
@@
 <wire x1="83.82" y1="55.88" x2="76.2" y2="55.88" width="0.1524" layer="91"/>
 <label x="78.74" y="55.88" size="1.778" layer="95"/>
+</segment>
+<segment>
+<pinref part="JP3" gate="A" pin="2"/>
+<wire x1="45.72" y1="17.78" x2="38.1" y2="17.78" width="0.1524" layer="91"/>
+<label x="38.1" y="17.78" size="1.778" layer="95"/>
+</segment>
+<segment>
+<pinref part="X1" gate="-1" pin="5"/>
+<wire x1="-20.32" y1="58.42" x2="-27.94" y2="58.42" width="0.1524" layer="91"/>
+<label x="-27.94" y="58.42" size="1.778" layer="95"/>
 </segment>
 </net>
@@
 </segment>
 </net>
+<net name="3V3" class="0">
+<segment>
+<pinref part="JP3" gate="A" pin="1"/>
+<wire x1="45.72" y1="20.32" x2="38.1" y2="20.32" width="0.1524" layer="91"/>
+<label x="38.1" y="20.32" size="1.778" layer="95"/>
+</segment>
+<segment>
+<pinref part="X1" gate="-1" pin="6"/>
+<wire x1="-27.94" y1="55.88" x2="-20.32" y2="55.88" width="0.1524" layer="91"/>
+<label x="-27.94" y="55.88" size="1.778" layer="95"/>
+</segment>
+</net>
+<net name="MISO" class="0">
+<segment>
+<pinref part="JP1" gate="A" pin="1"/>
+<wire x1="35.56" y1="55.88" x2="25.4" y2="55.88" width="0.1524" layer="91"/>
+<label x="22.86" y="55.88" size="1.778" layer="95"/>
+</segment>
+<segment>
+<pinref part="X1" gate="-1" pin="7"/>
+<wire x1="-27.94" y1="53.34" x2="-20.32" y2="53.34" width="0.1524" layer="91"/>
+<label x="-27.94" y="53.34" size="1.778" layer="95"/>
+</segment>
+</net>
+<net name="MOSI" class="0">
+<segment>
+<pinref part="JP1" gate="A" pin="4"/>
+<wire x1="43.18" y1="53.34" x2="55.88" y2="53.34" width="0.1524" layer="91"/>
+<label x="48.26" y="53.34" size="1.778" layer="95"/>
+</segment>
+<segment>
+<pinref part="X1" gate="-1" pin="3"/>
+<wire x1="-20.32" y1="63.5" x2="-27.94" y2="63.5" width="0.1524" layer="91"/>
+<label x="-27.94" y="63.5" size="1.778" layer="95"/>
+</segment>
+</net>
+<net name="SCLK" class="0">
+<segment>
+<pinref part="JP1" gate="A" pin="3"/>
+<wire x1="35.56" y1="53.34" x2="25.4" y2="53.34" width="0.1524" layer="91"/>
+<label x="22.86" y="53.34" size="1.778" layer="95"/>
+</segment>
+<segment>
+<pinref part="X1" gate="-1" pin="8"/>
+<wire x1="-27.94" y1="50.8" x2="-20.32" y2="50.8" width="0.1524" layer="91"/>
+<label x="-27.94" y="50.8" size="1.778" layer="95"/>
+</segment>
+</net>
+<net name="ACCEL2CS" class="0">
+<segment>
+<pinref part="JP1" gate="A" pin="5"/>
+<wire x1="35.56" y1="50.8" x2="25.4" y2="50.8" width="0.1524" layer="91"/>
+<label x="22.86" y="50.8" size="1.778" layer="95"/>
+</segment>
+<segment>
+<pinref part="X1" gate="-1" pin="4"/>
+<wire x1="-20.32" y1="60.96" x2="-27.94" y2="60.96" width="0.1524" layer="91"/>
+<label x="-27.94" y="60.96" size="1.778" layer="95"/>
+</segment>
+</net>
+<net name="TEMPBUS" class="0">
+<segment>
+<pinref part="JP2" gate="A" pin="1"/>
+<wire x1="45.72" y1="40.64" x2="35.56" y2="40.64" width="0.1524" layer="91"/>
+<label x="35.56" y="40.64" size="1.778" layer="95"/>
+</segment>
+<segment>
+<pinref part="X1" gate="-1" pin="10"/>
+<wire x1="2.54" y1="66.04" x2="-5.08" y2="66.04" width="0.1524" layer="91"/>
+<label x="-2.54" y="66.04" size="1.778" layer="95"/>
+</segment>
+</net>
+<net name="SDA" class="0">
+<segment>
+<pinref part="JP2" gate="A" pin="3"/>
+<wire x1="35.56" y1="38.1" x2="45.72" y2="38.1" width="0.1524" layer="91"/>
+<label x="35.56" y="38.1" size="1.778" layer="95"/>
+</segment>
+<segment>
+<pinref part="X1" gate="-1" pin="11"/>
+<wire x1="2.54" y1="63.5" x2="-5.08" y2="63.5" width="0.1524" layer="91"/>
+<label x="-2.54" y="63.5" size="1.778" layer="95"/>
+</segment>
+</net>
+<net name="SCL" class="0">
+<segment>
+<pinref part="JP2" gate="A" pin="5"/>
+<wire x1="35.56" y1="35.56" x2="45.72" y2="35.56" width="0.1524" layer="91"/>
+<label x="35.56" y="35.56" size="1.778" layer="95"/>
+</segment>
+<segment>
+<pinref part="X1" gate="-1" pin="12"/>
+<wire x1="2.54" y1="60.96" x2="-5.08" y2="60.96" width="0.1524" layer="91"/>
+<label x="-2.54" y="60.96" size="1.778" layer="95"/>
+</segment>
+</net>
+<net name="D46" class="0">
+<segment>
+<pinref part="JP2" gate="A" pin="2"/>
+<wire x1="63.5" y1="40.64" x2="53.34" y2="40.64" width="0.1524" layer="91"/>
+<label x="58.42" y="40.64" size="1.778" layer="95"/>
+</segment>
+<segment>
+<pinref part="X1" gate="-1" pin="13"/>
+<wire x1="2.54" y1="58.42" x2="-5.08" y2="58.42" width="0.1524" layer="91"/>
+<label x="-2.54" y="58.42" size="1.778" layer="95"/>
+</segment>
+</net>
+<net name="D47" class="0">
+<segment>
+<pinref part="JP2" gate="A" pin="4"/>
+<wire x1="63.5" y1="38.1" x2="53.34" y2="38.1" width="0.1524" layer="91"/>
+<label x="58.42" y="38.1" size="1.778" layer="95"/>
+</segment>
+<segment>
+<pinref part="X1" gate="-1" pin="14"/>
+<wire x1="2.54" y1="55.88" x2="-5.08" y2="55.88" width="0.1524" layer="91"/>
+<label x="-2.54" y="55.88" size="1.778" layer="95"/>
+</segment>
+</net>
+<net name="D48" class="0">
+<segment>
+<pinref part="JP2" gate="A" pin="6"/>
+<wire x1="63.5" y1="35.56" x2="53.34" y2="35.56" width="0.1524" layer="91"/>
+<label x="58.42" y="35.56" size="1.778" layer="95"/>
+</segment>
+<segment>
+<pinref part="X1" gate="-1" pin="15"/>
+<wire x1="2.54" y1="53.34" x2="-5.08" y2="53.34" width="0.1524" layer="91"/>
+<label x="-2.54" y="53.34" size="1.778" layer="95"/>
+</segment>
+</net>

Commit message: modified eagle boards and ordered.
Parts:
- removed BR: (no value), pinhead:PINHD-1X2
- removed JP2: (no value), pinhead:PINHD-2X3
- removed R2: 2.2K, rcl:R-US_0309/12
- added TEMP: (no value), pinhead:PINHD-1X3
- added U$5: RJ11V, RJ11V:RJ11V
- JP1: device pinhead:PINHD-2X3 -> pinhead:PINHD-1X5
- renumbered JP3 to DEBUG
Connections:
- removed net BR: BR.2, R2.2, U$1.P$2, U$2.P$5, U$3.P$2, U$4.P$5
- removed net D48: JP2.6, X1.15
- new net D45: JP1.3, X1.13
- net 3V3: now also U$5.P$6; no longer DEBUG.1
- net 5V: now also TEMP.2, U$1.P$2, U$2.P$5, U$3.P$2, U$4.P$5; no longer BR.1, JP1.2
- net ACCEL2CS: now also U$5.P$1; no longer JP1.5
- net D46: now also JP1.4, X1.14; no longer JP2.2, X1.13
- net D47: now also JP1.5, X1.15; no longer JP2.4, X1.14
- net GND: now also DEBUG.1, TEMP.1, U$5.P$5; no longer JP1.6, R2.1
- net MISO: now also U$5.P$4; no longer JP1.1
- net MOSI: now also U$5.P$3; no longer JP1.4
- net SCL: now also JP1.2; no longer JP2.5
- net SCLK: now also U$5.P$2; no longer JP1.3
- net SDA: now also JP1.1; no longer JP2.3
- net TEMPBUS: now also TEMP.3; no longer JP2.1
